Commit message: add vacuum_gripper link and gazebo_ros_vacuum_gripper_debugger plugin

File: universal_robot/ur_gazebo/urdf/ur.xacro (robot description, xacro)
@@ -73,3 +73,39 @@
     <origin xyz="0 0 0" rpy="0 0 0"/>
   </joint>
+   <!--vacuum_gripper joint and link define-->
+  <joint name="gripper_joint" type="fixed">
+    <origin xyz="0 0 0" rpy="0 3.14 1.571"/>
+    <parent link="tool0_controller"/>
+    <child link="vacuum_gripper"/>
+  </joint>
+  <link name="vacuum_gripper">
+    <visual>
+      <origin xyz="0 0 -0.025" rpy="0 0 0"/>
+      <geometry>
+        <cylinder radius="0.04" length="0.05"/>
+      </geometry>
+    </visual>
+    <collision>
+      <origin xyz="0 0 -0.025" rpy="0 0 0"/>
+      <geometry>
+        <cylinder radius="0.04" length="0.05"/>
+      </geometry>
+    </collision>
+    <inertial>
+      <mass value="1"/>
+      <origin xyz="0 0 0" rpy="0 0 0"/>
+      <inertia ixx="1e-04" ixy="0" ixz="0" iyy="1e-04" iyz="0" izz="1e-04"/>
+    </inertial>
+  </link>
+    <!-- Give cylinder properties to make it become an acutually vacuum_gripper -->
+  <gazebo>
+  <plugin name="gazebo_ros_vacuum_gripper_debugger" filename="libgazebo_ros_vacuum_gripper_debugger.so">
+      <robotNamespace>/vacuum_gripper</robotNamespace>
+      <bodyName>vacuum_gripper</bodyName>
+      <topicName>grasping</topicName>
+      <maxForce>200</maxForce>
+      <maxDistance>0.05</maxDistance>
+      <minDistance>0.01</minDistance>
+    </plugin>
+  </gazebo>
 </robot>

Commit message: move cylinder frame to rigtht position, and add start rviz script

File: universal_robot/ur_gazebo/urdf/ur.xacro (robot description, xacro)
@@ -75,5 +75,5 @@
    <!--vacuum_gripper joint and link define-->
   <joint name="gripper_joint" type="fixed">
-    <origin xyz="0 0 0" rpy="0 3.14 1.571"/>
+    <origin xyz="0 0 0.05" rpy="0 0 0"/>
     <parent link="tool0_controller"/>
     <child link="vacuum_gripper"/>

Commit message: 1. config movit and use position_controllers 2. modify path and copy world2 to moveit config folder 3. config new gazebo_ur10_robot in moveit 4. write the script to move robot to box position 5. use vaccum gripper ros service to turn on and grip (failed still debugging) 6. nex step: make vaccum gripper works and move it to the destination

File: universal_robot/ur_gazebo/urdf/ur.xacro (robot description, xacro)
@@ -1,4 +1,4 @@
 <?xml version="1.0"?>
-<robot xmlns:xacro="http://wiki.ros.org/xacro" name="$(arg robot_model)_robot">
+<robot xmlns:xacro="http://wiki.ros.org/xacro" name="ur10_robot">
   <!--
     This is a top-level xacro instantiating the Gazebo-specific version of the
@@ -26,8 +26,8 @@
   <xacro:include filename="$(find ur_gazebo)/urdf/ur_macro.xacro"/>
   <!--Declare arguments -->
-  <xacro:arg name="joint_limit_params" default=""/>
-  <xacro:arg name="physical_params" default=""/>
-  <xacro:arg name="kinematics_params" default=""/>
-  <xacro:arg name="visual_params" default=""/>
+  <xacro:arg name="joint_limit_params" default="$(find ur_description)/config/ur10/joint_limits.yaml"/>
+  <xacro:arg name="physical_params" default="$(find ur_description)/config/ur10/physical_parameters.yaml"/>
+  <xacro:arg name="kinematics_params" default="$(find ur_description)/config/ur10/default_kinematics.yaml"/>
+  <xacro:arg name="visual_params" default="$(find ur_description)/config/ur10/visual_parameters.yaml"/>
   <!--
     legal values:

File: vacuum_config/config/gazebo_ur10_robot.urdf (robot description, URDF)
Before this commit: robot ur10_robot, 11 links, 10 joints
Links:
- added link tool0_controller
- added link vacuum_gripper, mass 1; collision cylinder length=0.05 radius=0.04; visual cylinder length=0.05 radius=0.04
- added link world
Joints:
- added joint gripper_joint: type fixed, parent tool0_controller, child vacuum_gripper, origin xyz=0 0 0.055 rpy=0 0 0
- added joint tool_controller_fake_joint: type fixed, parent tool0, child tool0_controller, origin xyz=0 0 0 rpy=0 0 0
- added joint world_joint: type fixed, parent world, child base_link, origin xyz=0 0 0 rpy=0 0 0
- joint base_link-base_fixed_joint: child base_link -> base; parent base -> base_link
