Commit message: Update gripper joint and improve arm control precision: 1. Change `gripper_joint` type to revolute. 2. Add transmission for `gripper_joint` to prevent spinning. 3. Update world file to version 3. 4. Enhance arm control with precise positioning. 5. Increase sleep time for vacuum gripper stability before movement.

File: vacuum_config/config/gazebo_ur10_robot.urdf (robot description, URDF)
Before this commit: robot ur10_robot, 14 links, 13 joints
Joints:
- joint gripper_joint: axis (none) -> 0 0 1; limit (none) -> lower=-6.283185307179586 upper=6.283185307179586 effort=330.0 velocity=2.0943951023931953; type fixed -> revolute
